File: kicad/Lenovo_Keyboard.kicad_sch (KiCad schematic)
At the start: 5 parts, among them J1 Conn_01x34_Pin, J2 Conn_01x04_Socket, J3 Conn_01x04_Socket

Commit message: CapsLk/Escape LED support
Parts:
- removed J2: Conn_01x04_Socket, Connector_JST:JST_PH_S4B-PH-K_1x04_P2.00mm_Horizontal, symbol Connector:Conn_01x04_Socket
- removed J3: Conn_01x04_Socket, Connector_JST:JST_ZH_B4B-ZR_1x04_P1.50mm_Vertical, symbol Connector:Conn_01x04_Socket
- C1: value 10uF -> 0.1uF; footprint Capacitor_SMD:C_1206_3216Metric_Pad1.33x1.80mm_HandSolder -> Capacitor_SMD:C_0805_2012Metric_Pad1.18x1.45mm_HandSolder
Connections:
- net PFC_N0 is gone; now on net GND: J1.3 (Pin_3)
- net PFC_N2 is gone; now on net GND: J1.33 (Pin_33)
- net SCL is gone; now on net LED_ESC: A1.32 (GPIO27_ADC1)
- net SDA is gone; now on net LED_CAPSLK: A1.31 (GPIO26_ADC0)
- net PFC_N1 renamed LED_CAPSLK
- net PFC_N3 renamed LED_ESC
